File: side-markers-blinker.kicad_pcb (KiCad board)
At the start: 2 copper layers, 130 x 100 mm, 35 parts, among them J1 Conn_01x04_Socket, J2 Conn_01x02_Socket, J3 Conn_01x04_Socket, J4 Conn_01x02_Socket, Q1 IRF540N, Q2 BC546, Q3 BC546, Q4 IRF540N, Q5 BC546, Q6 BC546

Commit message: Add grid origin to kicad pcb.
Parts:
- moved H1 3.50 mm to (127.0, 82.5)
Other:
- board text added: "+"
- board text added: "-"
- board text added: "L+"
- board text added: "L-"
- board text added: "LB"
- board text added: "LS"
- board text added: "R+"
- board text added: "R-"
- board text added: "RB"
- board text added: "RS"
Changed lines of the file:
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@@
     )
     (pad_to_mask_clearance 0)
+    (grid_origin 127 82.5)
     (pcbplotparams
       (layerselection 0x00010fc_ffffffff)
@@
   )
   (footprint "MountingHole:MountingHole_6mm_Pad" (layer "F.Cu")
-    (at 130.5 82.5)
+    (at 127 82.5)
     (descr "Mounting Hole 6mm")
     (tags "mounting hole 6mm")
@@
   (gr_rect (start 62 32.5) (end 192 132.5)
     (stroke (width 0.1) (type default)) (fill none) (layer "Edge.Cuts"))
+  (gr_text "+" (at 70.5 54) (layer "F.SilkS")
+    (effects (font (size 1 1) (thickness 0.15)) (justify left bottom))
+  )
+  (gr_text "RB" (at 71.5 97.5 90) (layer "F.SilkS")
+    (effects (font (size 1 1) (thickness 0.15)) (justify left bottom))
+  )
+  (gr_text "RS" (at 71.5 106.5 90) (layer "F.SilkS")
+    (effects (font (size 1 1) (thickness 0.15)) (justify left bottom))
+  )
+  (gr_text "R+" (at 189.5 125 90) (layer "F.SilkS")
+    (effects (font (size 1 1) (thickness 0.15)) (justify left bottom))
+  )
+  (gr_text "+" (at 70.5 115) (layer "F.SilkS")
+    (effects (font (size 1 1) (thickness 0.15)) (justify left bottom))
+  )
+  (gr_text "-" (at 71.5 80.5 90) (layer "F.SilkS")
+    (effects (font (size 1 1) (thickness 0.15)) (justify left bottom))
+  )
+  (gr_text "R-" (at 189.5 116.5 90) (layer "F.SilkS")
+    (effects (font (size 1 1) (thickness 0.15)) (justify left bottom))
+  )
+  (gr_text "LS" (at 71.5 62.5 90) (layer "F.SilkS")
+    (effects (font (size 1 1) (thickness 0.15)) (justify left bottom))
+  )
+  (gr_text "-" (at 71.5 88.5 90) (layer "F.SilkS")
+    (effects (font (size 1 1) (thickness 0.15)) (justify left bottom))
+  )
+  (gr_text "L+" (at 190 41.5 90) (layer "F.SilkS")
+    (effects (font (size 1 1) (thickness 0.15)) (justify left bottom))
+  )
+  (gr_text "L-" (at 190 50.5 90) (layer "F.SilkS")
+    (effects (font (size 1 1) (thickness 0.15)) (justify left bottom))
+  )
+  (gr_text "LB" (at 71.5 72 90) (layer "F.SilkS")
+    (effects (font (size 1 1) (thickness 0.15)) (justify left bottom))
+  )
+  (dimension (type aligned) (layer "F.Cu")
+    (pts (xy 192 32.5) (xy 62 32.5))
+    (height 8)
+    (gr_text "130.0000 mm" (at 127 22.7) (layer "F.Cu")
+      (effects (font (size 1.5 1.5) (thickness 0.3)))
+    )
+    (format (prefix "") (suffix "") (units 3) (units_format 1) (precision 4))
+    (style (thickness 0.2) (arrow_length 1.27) (text_position_mode 0) (extension_height 0.58642) (extension_offset 0.5) keep_text_aligned)
+  )
+  (dimension (type aligned) (layer "F.Cu")
+    (pts (xy 195 32.5) (xy 195 132.5))
+    (height -16)
+    (gr_text "100.0000 mm" (at 209.2 82.5 90) (layer "F.Cu")
+      (effects (font (size 1.5 1.5) (thickness 0.3)))
+    )
+    (format (prefix "") (suffix "") (units 3) (units_format 1) (precision 4))
+    (style (thickness 0.2) (arrow_length 1.27) (text_position_mode 0) (extension_height 0.58642) (extension_offset 0.5) keep_text_aligned)
+  )
   (segment (start 117.968223 69.5) (end 117.891776 69.5) (width 1) (layer "F.Cu") (net 1))
   (segment (start 119.22 69.5) (end 122.426036 69.5) (width 1) (layer "F.Cu") (net 1))

Commit message: Reduce board size.
Parts:
- D1, D10, D2, D3, D4, D5, D6, D7, D8, D9: footprint Diode_THT:D_5W_P12.70mm_Horizontal -> Diode_THT:D_DO-41_SOD81_P7.62mm_Horizontal
- R1, R10, R11, R12, R2, R3, R4, R5, R6, R7, R8, R9: footprint Resistor_THT:R_Axial_DIN0411_L9.9mm_D3.6mm_P20.32mm_Horizontal -> Resistor_THT:R_Axial_DIN0207_L6.3mm_D2.5mm_P7.62mm_Horizontal
- moved J1 51.6 mm to (116.2, 95.0)
- moved J3 51.6 mm to (116.2, 103.0)
- moved D9 49.3 mm to (125.2, 104.4)
- moved R6 48.1 mm to (130.8, 104.4)
- moved D10 47.8 mm to (125.2, 93.6)
- moved R5 46.3 mm to (130.8, 93.6)
- moved D5 45.5 mm to (136.2, 104.4)
- moved D4 44.6 mm to (136.2, 93.6)
- moved H1 25.0 mm to (145.8, 99.0)
- moved J2 24.1 mm to (176.2, 72.0)
- moved Q4 22.3 mm to (151.1, 123.0)
- moved Q5 22.1 mm to (169.0, 92.2)
- moved Q6 22.1 mm to (169.0, 102.7)
- moved R9 21.9 mm to (148.3, 117.0)
- moved C2 20.0 mm to (127.3, 127.8)
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Routing:
- net Side marker lamp +24v R: track 0.00 -> 67.5 mm
- net Side marker lamp +24v L: track 0.00 -> 66.7 mm
- net AND gate: track 101.3 -> 48.8 mm
- net Side marker signal R: track 99.9 -> 50.4 mm, vias 0 -> 1
- net Side marker signal L: track 113.1 -> 70.7 mm
- net Net-(D5-A): track 41.7 -> 18.5 mm
- net Net-(Q4-G): track 32.9 -> 12.6 mm
- net Net-(Q1-G): track 33.3 -> 13.4 mm
- net Net-(D1-A): track 43.8 -> 25.3 mm
- net Net-(D6-K): track 21.8 -> 10.7 mm
- net Net-(D2-K): track 22.1 -> 11.2 mm
- net Net-(D1-K): track 34.0 -> 24.2 mm
- net Net-(D8-A): track 18.1 -> 9.48 mm
- net Net-(D7-K): track 32.9 -> 24.4 mm
- net Net-(D3-A): track 15.9 -> 10.2 mm
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- removed copper zone on F.Cu, net Side marker lamp +24v L
- removed copper zone on F.Cu, net Side marker lamp +24v R
Other:
- board size 130 x 100 mm -> 69 x 80.2 mm

Commit message: Remove unnecesary conections.
Parts:
- removed J1, J3: Conn_01x04_Socket, Connector_Wire:SolderWire-2.5sqmm_1x04_P8.8mm_D2.4mm_OD4.4mm
- removed J2, J4: Conn_01x02_Socket, Connector_Wire:SolderWire-2.5sqmm_1x02_P8.8mm_D2.4mm_OD4.4mm
- added J5: Conn_01x07_Socket, Connector_TE-Connectivity:TE_826576-7_1x07_P3.96mm_Vertical, F.Cu at (115.5, 111.0)
- moved H1 1.25 mm to (145.8, 97.8)
Routing:
- net Side marker lamp +24v R: track 67.5 -> 0.00 mm
- net Side marker lamp +24v L: track 66.7 -> 0.00 mm
- net Side marker lamp GND R: track 27.7 -> 85.0 mm, vias 0 -> 1
- net Side marker lamp GND L: track 27.2 -> 64.6 mm, vias 0 -> 1
- net Blinker signal L: track 9.09 -> 33.3 mm
- net Side marker signal L: track 70.7 -> 88.1 mm
- net Side marker signal R: track 50.4 -> 62.6 mm
- net Blinker signal R: track 9.09 -> 11.8 mm
Other:
- board size 69 x 80.2 mm -> 69 x 66.5 mm
- board text added: "GND"
- board text added: "out L"
- board text added: "out R"
- board text removed: "+"
- board text removed: "-"
- board text removed: "L+"
- board text removed: "L-"
- board text removed: "R+"
- board text removed: "R-"

Commit message: Redesigned pcb to use p channel mosfets.
Parts:
- removed J5: Conn_01x07_Socket, Connector_TE-Connectivity:TE_826576-7_1x07_P3.96mm_Vertical
- added J1: Conn_01x07_Socket, Connector_TE-Connectivity:TE_826576-7_1x07_P3.96mm_Vertical, F.Cu at (113.5, 108.1)
- added Q7: IRF4905, Package_TO_SOT_THT:TO-220-3_Horizontal_TabDown, F.Cu at (156.8, 110.3)
- added Q8: IRF4905, Package_TO_SOT_THT:TO-220-3_Horizontal_TabDown, F.Cu at (156.2, 77.1)
- added R13: 10k, Resistor_THT:R_Axial_DIN0207_L6.3mm_D2.5mm_P7.62mm_Horizontal, F.Cu at (163.6, 72.7)
- added R14: 10k, Resistor_THT:R_Axial_DIN0207_L6.3mm_D2.5mm_P7.62mm_Horizontal, F.Cu at (163.6, 69.5)
- C1, C2: footprint Capacitor_THT:CP_Radial_D4.0mm_P1.50mm -> Capacitor_THT:CP_Radial_D5.0mm_P2.00mm
- Q1, Q4: value IRF540N -> BC547; footprint Package_TO_SOT_THT:TO-220-3_Horizontal_TabDown -> Package_TO_SOT_THT:TO-92_Inline
- Q2, Q3, Q5, Q6: value BC546 -> BC547
- R1, R10: value 100k -> 10k
- R11, R12, R5, R6: value 1k -> 10k
- R2, R9: value 50k -> 10k
- moved R1 55.7 mm to (124.8, 111.6), turned to 90 degrees
- moved C2 55.1 mm to (122.8, 72.8)
- moved Q1 49.5 mm to (133.0, 120.8)
- moved D1 45.4 mm to (120.0, 111.8), turned to 90 degrees
- moved D6 44.7 mm to (127.2, 77.8), turned to 0 degrees
- moved R10 43.2 mm to (144.8, 76.3), turned to 90 degrees
- moved C1 42.7 mm to (117.8, 121.2)
- moved Q6 39.0 mm to (148.8, 69.3)
- moved D3 38.9 mm to (129.5, 111.8), turned to 90 degrees
- moved Q3 36.8 mm to (157.6, 92.0)
- moved R3 35.7 mm to (139.5, 103.9), turned to -90 degrees
- moved Q5 35.5 mm to (148.2, 121.0)
- moved R7 34.5 mm to (151.6, 85.6), turned to -90 degrees
- moved D8 33.1 mm to (134.4, 89.2), turned to -90 degrees
- moved R2 31.9 mm to (124.8, 89.2), turned to -90 degrees
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Connections:
- C1 pad 1: Net-(D2-K) -> Net-(D5-K)
- D1 pad 2: Net-(D1-A) -> Blinker signal R input
- D10 pad 2: Blinker signal L -> Net-(D10-A)
- D2 pad 2: Net-(D1-A) -> Blinker signal L input
- D3 pad 1: Net-(D1-K) -> AND gate
- D4 pad 2: Net-(D1-A) -> Net-(D4-A)
- D5 pad 1: AND gate -> Net-(D5-K)
- D5 pad 2: Net-(D5-A) -> Net-(D3-A)
- D6 pad 2: Net-(D5-A) -> Net-(D4-A)
- D7 pad 2: Net-(D5-A) -> Net-(D3-A)
- D8 pad 1: Net-(D7-K) -> Net-(D10-K)
- D8 pad 2: Net-(D8-A) -> Net-(D4-A)
- D9 pad 1: Net-(D9-K) -> Net-(D7-K)
- D9 pad 2: Blinker signal R -> Net-(D9-A)
- Q1 pad 1: Net-(Q1-G) -> Net-(D9-A)
- Q1 pad 2: Side marker lamp GND L -> Net-(Q1-B)
- Q2 pad 1: Net-(D3-A) -> Net-(D10-A)
- Q3 pad 1: Net-(D8-A) -> AND gate
- Q3 pad 3: GND -> Net-(Q3-E)
- Q4 pad 1: Net-(Q4-G) -> Net-(Q3-E)
- Q4 pad 2: Side marker lamp GND R -> Net-(Q4-B)
- Q5 pad 1: AND gate -> Net-(Q5-C)
- Q5 pad 3: Net-(Q5-E) -> GND
- Q6 pad 1: Net-(Q5-E) -> Net-(Q6-C)
- R1 pad 1: Net-(Q1-G) -> Net-(D1-K)
- R1 pad 2: GND -> Net-(D3-A)
- R10 pad 1: Net-(Q4-G) -> Net-(D10-K)
- R10 pad 2: GND -> Net-(Q6-B)
- R11 pad 1: Side marker signal L -> Net-(Q7-G)
- R11 pad 2: Net-(Q5-B) -> +24v when igniton on
- R12 pad 1: Side marker signal R -> Net-(Q7-G)
- R12 pad 2: Net-(Q6-B) -> Net-(Q5-C)
- R2 pad 1: Net-(D1-K) -> Net-(D2-K)
- R2 pad 2: Net-(Q1-G) -> Net-(D4-A)
- R3 pad 1: Side marker signal L -> Side markers signal input
- R3 pad 2: Net-(D3-A) -> Net-(D9-A)
- R4 pad 1: Net-(D2-K) -> Side markers signal input
- R4 pad 2: Net-(Q2-B) -> Net-(D10-A)
- R5 pad 1: Net-(D10-K) -> Net-(D5-K)
- R5 pad 2: Net-(D1-A) -> Net-(Q1-B)
- R6 pad 1: Net-(D9-K) -> Net-(D6-K)
- R6 pad 2: Net-(D5-A) -> Net-(Q2-B)
- R7 pad 1: Side marker signal R -> Blinker signal R input
- R7 pad 2: Net-(D8-A) -> Net-(Q3-B)
- R8 pad 1: Net-(D6-K) -> Blinker signal L input
- R8 pad 2: Net-(Q3-B) -> Net-(Q4-B)
- R9 pad 2: Net-(Q4-G) -> Net-(Q5-B)
Routing:
- net Side marker signal L: track 88.1 -> 0.00 mm, vias 1 -> 0
- net Side marker lamp GND R: track 85.0 -> 0.00 mm, vias 1 -> 0
- net Blinker signal R input: track 0.00 -> 73.1 mm
- net Side marker lamp GND L: track 64.6 -> 0.00 mm, vias 1 -> 0
- net Side marker lamp +24 R output: track 0.00 -> 63.5 mm
- net Side marker signal R: track 62.6 -> 0.00 mm, vias 1 -> 0
- net Side marker lamp +24 L output: track 0.00 -> 49.2 mm
- net Side markers signal input: track 0.00 -> 49.2 mm
- net Blinker signal L input: track 0.00 -> 43.2 mm
- net Blinker signal L: track 33.3 -> 0.00 mm
- net Net-(D4-A): track 0.00 -> 30.3 mm
- net Net-(D1-A): track 25.3 -> 0.00 mm
- net Net-(D1-K): track 24.2 -> 4.83 mm
- net Net-(D10-A): track 0.00 -> 18.9 mm
- net Net-(D5-A): track 18.5 -> 0.00 mm
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- added copper zone on F.Cu, net +24v when igniton on
Other:
- board text removed: "GND"
- board text removed: "LB"
- board text removed: "LS"
- board text removed: "RB"
- board text removed: "RS"
- board text removed: "out L"
- board text removed: "out R"

Commit message: Fixed mosfet connection.
Connections:
- Q7 pad 2: +24v when igniton on -> Side marker lamp +24 R output
- Q7 pad 3: Side marker lamp +24 R output -> +24v when igniton on
- Q8 pad 2: +24v when igniton on -> Side marker lamp +24 L output
- Q8 pad 3: Side marker lamp +24 L output -> +24v when igniton on
Routing:
- net +24v when igniton on: track 0.00 -> 19.1 mm
- net Side marker lamp +24 R output: track 63.5 -> 76.5 mm
- net Side marker lamp +24 L output: track 49.2 -> 50.2 mm
Changed lines of the file:
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@@
       (net 29 "Net-(Q7-G)") (pinfunction "G") (pintype "input"))
     (pad "2" thru_hole oval (at 2.54 0 270) (size 1.905 2) (drill 1.1) (layers "*.Cu" "*.Mask")
-      (net 18 "+24v when igniton on") (pinfunction "D") (pintype "passive"))
+      (net 16 "Side marker lamp +24 R output") (pinfunction "D") (pintype "passive"))
     (pad "3" thru_hole oval (at 5.08 0 270) (size 1.905 2) (drill 1.1) (layers "*.Cu" "*.Mask")
-      (net 16 "Side marker lamp +24 R output") (pinfunction "S") (pintype "passive"))
+      (net 18 "+24v when igniton on") (pinfunction "S") (pintype "passive"))
     (model "${KICAD6_3DMODEL_DIR}/Package_TO_SOT_THT.3dshapes/TO-220-3_Horizontal_TabDown.wrl"
       (offset (xyz 0 0 0))
@@
       (net 21 "Net-(Q8-G)") (pinfunction "G") (pintype "input"))
     (pad "2" thru_hole oval (at 2.54 0 270) (size 1.905 2) (drill 1.1) (layers "*.Cu" "*.Mask")
-      (net 18 "+24v when igniton on") (pinfunction "D") (pintype "passive"))
+      (net 17 "Side marker lamp +24 L output") (pinfunction "D") (pintype "passive"))
     (pad "3" thru_hole oval (at 5.08 0 270) (size 1.905 2) (drill 1.1) (layers "*.Cu" "*.Mask")
-      (net 17 "Side marker lamp +24 L output") (pinfunction "S") (pintype "passive"))
+      (net 18 "+24v when igniton on") (pinfunction "S") (pintype "passive"))
     (model "${KICAD6_3DMODEL_DIR}/Package_TO_SOT_THT.3dshapes/TO-220-3_Horizontal_TabDown.wrl"
       (offset (xyz 0 0 0))
@@
   (segment (start 118.6001 91.0841) (end 137.1759 91.0841) (width 1) (layer "F.Cu") (net 15))
   (segment (start 117.9003 90.3843) (end 118.6001 91.0841) (width 1) (layer "F.Cu") (net 15))
-  (segment (start 145.6 108.65) (end 125.4 108.65) (width 2) (layer "F.Cu") (net 16))
-  (segment (start 155.2 118.65) (end 152 118.65) (width 2) (layer "F.Cu") (net 16))
-  (segment (start 116.8 98.45) (end 116.8 93.65) (width 2) (layer "F.Cu") (net 16))
-  (segment (start 149 115.65) (end 149 112.05) (width 2) (layer "F.Cu") (net 16))
-  (segment (start 120.2 100.05) (end 118.4 100.05) (width 2) (layer "F.Cu") (net 16))
-  (segment (start 152 118.65) (end 149 115.65) (width 2) (layer "F.Cu") (net 16))
-  (segment (start 156.77 115.39) (end 156.77 117.08) (width 2) (layer "F.Cu") (net 16))
-  (segment (start 122.4 105.65) (end 122.4 102.25) (width 2) (layer "F.Cu") (net 16))
-  (segment (start 125.4 108.65) (end 122.4 105.65) (width 2) (layer "F.Cu") (net 16))
-  (segment (start 115.44 92.29) (end 113.4825 92.29) (width 2) (layer "F.Cu") (net 16))
-  (segment (start 116.8 93.65) (end 115.44 92.29) (width 2) (layer "F.Cu") (net 16))
-  (segment (start 149 112.05) (end 145.6 108.65) (width 2) (layer "F.Cu") (net 16))
-  (segment (start 118.4 100.05) (end 116.8 98.45) (width 2) (layer "F.Cu") (net 16))
-  (segment (start 122.4 102.25) (end 120.2 100.05) (width 2) (layer "F.Cu") (net 16))
-  (segment (start 156.77 117.08) (end 155.2 118.65) (width 2) (layer "F.Cu") (net 16))
-  (segment (start 143.34 82.19) (end 156.17 82.19) (width 2) (layer "F.Cu") (net 17))
-  (segment (start 142 80.85) (end 143.34 82.19) (width 2) (layer "F.Cu") (net 17))
-  (segment (start 115.32 88.33) (end 121 82.65) (width 2) (layer "F.Cu") (net 17))
-  (segment (start 133.8 82.65) (end 138.2 78.25) (width 2) (layer "F.Cu") (net 17))
-  (segment (start 113.4825 88.33) (end 115.32 88.33) (width 2) (layer "F.Cu") (net 17))
-  (segment (start 142 79.65) (end 142 80.85) (width 2) (layer "F.Cu") (net 17))
-  (segment (start 121 82.65) (end 133.8 82.65) (width 2) (layer "F.Cu") (net 17))
-  (segment (start 140.6 78.25) (end 142 79.65) (width 2) (layer "F.Cu") (net 17))
-  (segment (start 138.2 78.25) (end 140.6 78.25) (width 2) (layer "F.Cu") (net 17))
+  (segment (start 162 117.65) (end 162 114.65) (width 2) (layer "F.Cu") (net 16))
+  (segment (start 159.6 120.05) (end 162 117.65) (width 2) (layer "F.Cu") (net 16))
+  (segment (start 145.6 108.65) (end 149.8 112.85) (width 2) (layer "F.Cu") (net 16))
+  (segment (start 120.2 100.05) (end 122.4 102.25) (width 2) (layer "F.Cu") (net 16))
+  (segment (start 122.4 105.65) (end 125.4 108.65) (width 2) (layer "F.Cu") (net 16))
+  (segment (start 162 114.65) (end 160.2 112.85) (width 2) (layer "F.Cu") (net 16))
+  (segment (start 118.4 100.05) (end 120.2 100.05) (width 2) (layer "F.Cu") (net 16))
+  (segment (start 160.2 112.85) (end 156.77 112.85) (width 2) (layer "F.Cu") (net 16))
+  (segment (start 154 120.05) (end 159.6 120.05) (width 2) (layer "F.Cu") (net 16))
+  (segment (start 122.4 102.25) (end 122.4 105.65) (width 2) (layer "F.Cu") (net 16))
+  (segment (start 116.8 98.45) (end 118.4 100.05) (width 2) (layer "F.Cu") (net 16))
+  (segment (start 125.4 108.65) (end 145.6 108.65) (width 2) (layer "F.Cu") (net 16))
+  (segment (start 149.8 115.85) (end 154 120.05) (width 2) (layer "F.Cu") (net 16))
+  (segment (start 116.8 93.65) (end 116.8 98.45) (width 2) (layer "F.Cu") (net 16))
+  (segment (start 113.4825 92.29) (end 115.44 92.29) (width 2) (layer "F.Cu") (net 16))
+  (segment (start 115.44 92.29) (end 116.8 93.65) (width 2) (layer "F.Cu") (net 16))
+  (segment (start 149.8 112.85) (end 149.8 115.85) (width 2) (layer "F.Cu") (net 16))
+  (segment (start 142 80.85) (end 142 79.65) (width 2) (layer "F.Cu") (net 17))
+  (segment (start 146.86 82.19) (end 143.34 82.19) (width 2) (layer "F.Cu") (net 17))
+  (segment (start 143.34 82.19) (end 142 80.85) (width 2) (layer "F.Cu") (net 17))
+  (segment (start 156.17 79.65) (end 149.4 79.65) (width 2) (layer "F.Cu") (net 17))
+  (segment (start 138.2 78.25) (end 133.8 82.65) (width 2) (layer "F.Cu") (net 17))
+  (segment (start 142 79.65) (end 140.6 78.25) (width 2) (layer "F.Cu") (net 17))
+  (segment (start 140.6 78.25) (end 138.2 78.25) (width 2) (layer "F.Cu") (net 17))
+  (segment (start 133.8 82.65) (end 121 82.65) (width 2) (layer "F.Cu") (net 17))
+  (segment (start 115.32 88.33) (end 113.4825 88.33) (width 2) (layer "F.Cu") (net 17))
+  (segment (start 121 82.65) (end 115.32 88.33) (width 2) (layer "F.Cu") (net 17))
+  (segment (start 149.4 79.65) (end 146.86 82.19) (width 2) (layer "F.Cu") (net 17))
+  (segment (start 156.77 115.39) (end 156.35 115.39) (width 1) (layer "F.Cu") (net 18))
+  (segment (start 156.35 115.39) (end 153.41 112.45) (width 1) (layer "F.Cu") (net 18))
+  (segment (start 152.4 74.65) (end 152.4 80.05) (width 1) (layer "B.Cu") (net 18))
+  (segment (start 154.54 82.19) (end 156.17 82.19) (width 1) (layer "B.Cu") (net 18))
+  (segment (start 152.4 80.05) (end 154.54 82.19) (width 1) (layer "B.Cu") (net 18))
+  (segment (start 154.4 72.65) (end 152.4 74.65) (width 1) (layer "B.Cu") (net 18))
+  (segment (start 155.99 72.65) (end 154.4 72.65) (width 1) (layer "B.Cu") (net 18))
   (segment (start 133.04 122.05) (end 129.61 122.05) (width 1) (layer "F.Cu") (net 19))
   (segment (start 155.88 101.64) (end 155.89 101.65) (width 1) (layer "F.Cu") (net 20))
