File: side-markers-blinker.kicad_sch (KiCad schematic)
At the start: 35 parts, among them J1 Conn_01x04_Socket, J2 Conn_01x02_Socket, J3 Conn_01x04_Socket, J4 Conn_01x02_Socket, Q1 IRF540N, Q2 BC546, Q3 BC546, Q4 IRF540N, Q5 BC546, Q6 BC546

Commit message: Reduce board size.
Parts:
- D1, D10, D2, D3, D4, D5, D6, D7, D8, D9: footprint Diode_THT:D_5W_P12.70mm_Horizontal -> Diode_THT:D_DO-41_SOD81_P7.62mm_Horizontal
- R1, R10, R11, R12, R2, R3, R4, R5, R6, R7, R8, R9: footprint Resistor_THT:R_Axial_DIN0411_L9.9mm_D3.6mm_P20.32mm_Horizontal -> Resistor_THT:R_Axial_DIN0207_L6.3mm_D2.5mm_P7.62mm_Horizontal
Changed lines of the file:
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@@
       (effects (font (size 1.27 1.27)) (justify right))
     )
-    (property "Footprint" "Diode_THT:D_5W_P12.70mm_Horizontal" (at 123.19 33.02 90)
+    (property "Footprint" "Diode_THT:D_DO-41_SOD81_P7.62mm_Horizontal" (at 123.19 33.02 90)
       (effects (font (size 1.27 1.27)) hide)
     )
@@
       (effects (font (size 1.27 1.27)))
     )
-    (property "Footprint" "Resistor_THT:R_Axial_DIN0411_L9.9mm_D3.6mm_P20.32mm_Horizontal" (at 114.3 27.94 0)
+    (property "Footprint" "Resistor_THT:R_Axial_DIN0207_L6.3mm_D2.5mm_P7.62mm_Horizontal" (at 114.3 27.94 0)
       (effects (font (size 1.27 1.27)) hide)
     )
@@
       (effects (font (size 1.27 1.27)))
     )
-    (property "Footprint" "Resistor_THT:R_Axial_DIN0411_L9.9mm_D3.6mm_P20.32mm_Horizontal" (at 119.38 115.57 0)
+    (property "Footprint" "Resistor_THT:R_Axial_DIN0207_L6.3mm_D2.5mm_P7.62mm_Horizontal" (at 119.38 115.57 0)
       (effects (font (size 1.27 1.27)) hide)
     )
@@
       (effects (font (size 1.27 1.27)))
     )
-    (property "Footprint" "Resistor_THT:R_Axial_DIN0411_L9.9mm_D3.6mm_P20.32mm_Horizontal" (at 135.89 102.87 0)
+    (property "Footprint" "Resistor_THT:R_Axial_DIN0207_L6.3mm_D2.5mm_P7.62mm_Horizontal" (at 135.89 102.87 0)
       (effects (font (size 1.27 1.27)) hide)
     )
@@
       (effects (font (size 1.27 1.27)))
     )
-    (property "Footprint" "Resistor_THT:R_Axial_DIN0411_L9.9mm_D3.6mm_P20.32mm_Horizontal" (at 116.84 50.8 0)
+    (property "Footprint" "Resistor_THT:R_Axial_DIN0207_L6.3mm_D2.5mm_P7.62mm_Horizontal" (at 116.84 50.8 0)
       (effects (font (size 1.27 1.27)) hide)
     )
@@
       (effects (font (size 1.27 1.27)) (justify right))
     )
-    (property "Footprint" "Diode_THT:D_5W_P12.70mm_Horizontal" (at 93.98 102.87 90)
+    (property "Footprint" "Diode_THT:D_DO-41_SOD81_P7.62mm_Horizontal" (at 93.98 102.87 90)
       (effects (font (size 1.27 1.27)) hide)
     )
@@
       (effects (font (size 1.27 1.27)) (justify right))
     )
-    (property "Footprint" "Diode_THT:D_5W_P12.70mm_Horizontal" (at 115.57 107.95 90)
+    (property "Footprint" "Diode_THT:D_DO-41_SOD81_P7.62mm_Horizontal" (at 115.57 107.95 90)
       (effects (font (size 1.27 1.27)) hide)
     )
@@
       (effects (font (size 1.27 1.27)))
     )
-    (property "Footprint" "Resistor_THT:R_Axial_DIN0411_L9.9mm_D3.6mm_P20.32mm_Horizontal" (at 60.96 170.18 0)
+    (property "Footprint" "Resistor_THT:R_Axial_DIN0207_L6.3mm_D2.5mm_P7.62mm_Horizontal" (at 60.96 170.18 0)
       (effects (font (size 1.27 1.27)) hide)
     )
@@
       (effects (font (size 1.27 1.27)))
     )
-    (property "Footprint" "Resistor_THT:R_Axial_DIN0411_L9.9mm_D3.6mm_P20.32mm_Horizontal" (at 99.06 38.1 0)
+    (property "Footprint" "Resistor_THT:R_Axial_DIN0207_L6.3mm_D2.5mm_P7.62mm_Horizontal" (at 99.06 38.1 0)
       (effects (font (size 1.27 1.27)) hide)
     )
@@
       (effects (font (size 1.27 1.27)))
     )
-    (property "Footprint" "Resistor_THT:R_Axial_DIN0411_L9.9mm_D3.6mm_P20.32mm_Horizontal" (at 60.96 156.21 0)
+    (property "Footprint" "Resistor_THT:R_Axial_DIN0207_L6.3mm_D2.5mm_P7.62mm_Horizontal" (at 60.96 156.21 0)
       (effects (font (size 1.27 1.27)) hide)
     )
@@
       (effects (font (size 1.27 1.27)) (justify left))
     )
-    (property "Footprint" "Resistor_THT:R_Axial_DIN0411_L9.9mm_D3.6mm_P20.32mm_Horizontal" (at 144.78 106.68 0)
+    (property "Footprint" "Resistor_THT:R_Axial_DIN0207_L6.3mm_D2.5mm_P7.62mm_Horizontal" (at 144.78 106.68 0)
       (effects (font (size 1.27 1.27)) hide)
     )
@@
       (effects (font (size 1.27 1.27)))
     )
-    (property "Footprint" "Resistor_THT:R_Axial_DIN0411_L9.9mm_D3.6mm_P20.32mm_Horizontal" (at 133.35 38.1 0)
+    (property "Footprint" "Resistor_THT:R_Axial_DIN0207_L6.3mm_D2.5mm_P7.62mm_Horizontal" (at 133.35 38.1 0)
       (effects (font (size 1.27 1.27)) hide)
     )
@@
       (effects (font (size 1.27 1.27)) (justify right))
     )
-    (property "Footprint" "Diode_THT:D_5W_P12.70mm_Horizontal" (at 91.44 38.1 90)
+    (property "Footprint" "Diode_THT:D_DO-41_SOD81_P7.62mm_Horizontal" (at 91.44 38.1 90)
       (effects (font (size 1.27 1.27)) hide)
     )
@@
       (effects (font (size 1.27 1.27)))
     )
-    (property "Footprint" "Diode_THT:D_5W_P12.70mm_Horizontal" (at 119.38 102.87 90)
+    (property "Footprint" "Diode_THT:D_DO-41_SOD81_P7.62mm_Horizontal" (at 119.38 102.87 90)
       (effects (font (size 1.27 1.27)) hide)
     )
@@
       (effects (font (size 1.27 1.27)))
     )
-    (property "Footprint" "Resistor_THT:R_Axial_DIN0411_L9.9mm_D3.6mm_P20.32mm_Horizontal" (at 101.6 102.87 0)
+    (property "Footprint" "Resistor_THT:R_Axial_DIN0207_L6.3mm_D2.5mm_P7.62mm_Horizontal" (at 101.6 102.87 0)
       (effects (font (size 1.27 1.27)) hide)
     )
@@
       (effects (font (size 1.27 1.27)))
     )
-    (property "Footprint" "Resistor_THT:R_Axial_DIN0411_L9.9mm_D3.6mm_P20.32mm_Horizontal" (at 116.84 92.71 0)
+    (property "Footprint" "Resistor_THT:R_Axial_DIN0207_L6.3mm_D2.5mm_P7.62mm_Horizontal" (at 116.84 92.71 0)
       (effects (font (size 1.27 1.27)) hide)
     )
@@
       (effects (font (size 1.27 1.27)) (justify right))
     )
-    (property "Footprint" "Diode_THT:D_5W_P12.70mm_Horizontal" (at 125.73 97.79 90)
+    (property "Footprint" "Diode_THT:D_DO-41_SOD81_P7.62mm_Horizontal" (at 125.73 97.79 90)
       (effects (font (size 1.27 1.27)) hide)
     )
@@
       (effects (font (size 1.27 1.27)) (justify right))
     )
-    (property "Footprint" "Diode_THT:D_5W_P12.70mm_Horizontal" (at 101.6 45.72 90)
+    (property "Footprint" "Diode_THT:D_DO-41_SOD81_P7.62mm_Horizontal" (at 101.6 45.72 90)
       (effects (font (size 1.27 1.27)) hide)
     )
@@
       (effects (font (size 1.27 1.27)) (justify right))
     )
-    (property "Footprint" "Diode_THT:D_5W_P12.70mm_Horizontal" (at 104.14 110.49 90)
+    (property "Footprint" "Diode_THT:D_DO-41_SOD81_P7.62mm_Horizontal" (at 104.14 110.49 90)
       (effects (font (size 1.27 1.27)) hide)
     )
@@
       (effects (font (size 1.27 1.27)) (justify left))
     )
-    (property "Footprint" "Resistor_THT:R_Axial_DIN0411_L9.9mm_D3.6mm_P20.32mm_Horizontal" (at 142.24 41.91 0)
+    (property "Footprint" "Resistor_THT:R_Axial_DIN0207_L6.3mm_D2.5mm_P7.62mm_Horizontal" (at 142.24 41.91 0)
       (effects (font (size 1.27 1.27)) hide)
     )
@@
       (effects (font (size 1.27 1.27)) (justify right))
     )
-    (property "Footprint" "Diode_THT:D_5W_P12.70mm_Horizontal" (at 113.03 43.18 90)
+    (property "Footprint" "Diode_THT:D_DO-41_SOD81_P7.62mm_Horizontal" (at 113.03 43.18 90)
       (effects (font (size 1.27 1.27)) hide)
     )
@@
       (effects (font (size 1.27 1.27)))
     )
-    (property "Footprint" "Diode_THT:D_5W_P12.70mm_Horizontal" (at 116.84 38.1 90)
-      (effects (font (size 1.27 1.27)) hide)
-    )
+    (property "Footprint" "Diode_THT:D_DO-41_SOD81_P7.62mm_Horizontal" (at 116.84 38.1 90)
+      (effects (font (size 1.27 1.27)) hide)
+    )

Commit message: Remove unnecesary conections.
Parts:
- removed J1, J3: Conn_01x04_Socket, Connector_Wire:SolderWire-2.5sqmm_1x04_P8.8mm_D2.4mm_OD4.4mm, symbol Connector:Conn_01x04_Socket
- removed J2, J4: Conn_01x02_Socket, Connector_Wire:SolderWire-2.5sqmm_1x02_P8.8mm_D2.4mm_OD4.4mm, symbol Connector:Conn_01x02_Socket
- added J5: Conn_01x07_Socket, Connector_TE-Connectivity:TE_826576-7_1x07_P3.96mm_Vertical, symbol Connector:Conn_01x07_Socket
Connections:
- net Blinker signal L: now also J5.4 (Pin_4)
- net Blinker signal R: now also J5.2 (Pin_2)
- net GND: now also J5.1 (Pin_1)
- net Side marker lamp GND L: now also J5.7 (Pin_7)
- net Side marker lamp GND R: now also J5.6 (Pin_6)
- net Side marker signal L: now also J5.5 (Pin_5)
- net Side marker signal R: now also J5.3 (Pin_3)
Other:
- moved on the sheet: C1, C2, D1, D10, D2, D3, D4, D5, D6, D7, D8, D9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

Commit message: Redesigned pcb to use p channel mosfets.
Parts:
- removed D5, D7, D9: ~, Diode_THT:D_DO-41_SOD81_P7.62mm_Horizontal, symbol Device:D_Small
- removed Q1, Q4: IRF540N, Package_TO_SOT_THT:TO-220-3_Horizontal_TabDown, symbol Transistor_FET:IRF540N
- removed Q2, Q3, Q5, Q6: BC546, Package_TO_SOT_THT:TO-92_Inline, symbol Transistor_BJT:BC546
- removed R7, R8: 10k, Resistor_THT:R_Axial_DIN0207_L6.3mm_D2.5mm_P7.62mm_Horizontal, symbol Device:R_Small
- added D10, D2, D4: ~, Diode_THT:D_DO-41_SOD81_P7.62mm_Horizontal, symbol Device:D_Small
- added Q1, Q2, Q3, Q4, Q5, Q6: BC547, Package_TO_SOT_THT:TO-92_Inline, symbol Transistor_BJT:BC547
- added Q7, Q8: IRF4905, Package_TO_SOT_THT:TO-220-3_Horizontal_TabDown, symbol Transistor_FET:IRF4905
- added R13, R14, R2, R4: 10k, Resistor_THT:R_Axial_DIN0207_L6.3mm_D2.5mm_P7.62mm_Horizontal, symbol Device:R_Small
- C1, C2: footprint Capacitor_THT:CP_Radial_D4.0mm_P1.50mm -> Capacitor_THT:CP_Radial_D5.0mm_P2.00mm
- R1: renamed from R5; value 1k -> 10k
- R10: value 100k -> 10k
- R11: renamed from R2; value 50k -> 10k
- R12: renamed from R1; value 100k -> 10k
- R6: value 1k -> 10k
- R7: renamed from R11; value 1k -> 10k
- R8: renamed from R12; value 1k -> 10k
- R9: value 50k -> 10k
- renumbered D10 to D1, D4 to D3, D2 to D5, D1 to D7, D3 to D9, J5 to J1, R4 to R5
Connections:
- net Blinker signal R is gone; now on net Blinker signal R input: J1.2 (Pin_2)
- net AND gate: now also D4.1 (K), Q3.1 (C)
- net GND: now also Q1.3 (E), Q2.3 (E), Q4.3 (E), Q5.3 (E), Q6.3 (E); no longer R10.2, R12.2
- net at R10.1: now also D8.1 (K), D10.1 (K); no longer R9.2
- net at R7.2: now also Q3.2 (B)
- net at D7.1 (K), D9.1 (K): now also R9.1; no longer R11.1
- net at D9.2 (A), R3.2: now also Q1.1 (C)
- net at R8.2: now also Q4.2 (B)
- net at C2.1, D6.1 (K): now also R6.1
- net at D8.2 (A): now also D6.2 (A), D4.2 (A), R2.2
- net at R5.2: now also Q1.2 (B)
- net at R12.1: now also R11.1, Q7.1 (G); no longer R11.2
- net at R6.2: now also Q2.2 (B); no longer D6.2 (A)
- net Blinker signal L renamed Blinker signal R input
- net Blinker signal R input: now also R7.1; no longer J1.4 (Pin_4)
- net Side marker lamp GND L renamed +24v when igniton on
- net +24v when igniton on: now also R11.2, Q7.2 (D), Q8.2 (D), R13.2
- net Side marker lamp GND R renamed Side marker lamp +24 L output
- net Side marker lamp +24 L output: now also Q8.3 (S)
- removed net Side marker signal L: J1.5 (Pin_5), R3.1, R7.1
- net Side marker signal R renamed Blinker signal L input
- net Blinker signal L input: now also D2.2 (A)
- new net: Q8.1 (G), R13.1, R14.1
- new net: D10.2 (A), Q2.1 (C), R4.2
- new net: Q6.2 (B), R10.2
- new net: Q3.3 (E), Q4.1 (C)
- new net: Q6.1 (C), R14.2
- new net: Q5.2 (B), R9.2
- new net: Q5.1 (C), R12.2
- new net: D2.1 (K), R2.1
- new net Side marker lamp +24 R output: J1.5 (Pin_5), Q7.3 (S)
- new net Side markers signal input: J1.4 (Pin_4), R3.1, R4.1
Other:
- moved on the sheet: R11, R12, R3

Commit message: Updated schematic.
Other:
- note added: "AND gate"
- note added: "Connectors"
- note added: "Left side circuit"
- note added: "Right side circuit"
- moved on the sheet: C1, C2, D1, D10, D2, D3, D4, D5, D6, D7, D8, D9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

Commit message: Fixed mosfet connection.
Connections:
- net +24v when igniton on: now also Q7.3 (S), Q8.3 (S); no longer Q7.2 (D), Q8.2 (D)
- net Side marker lamp +24 L output: now also Q8.2 (D); no longer Q8.3 (S)
- net Side marker lamp +24 R output: now also Q7.2 (D); no longer Q7.3 (S)
Changed lines of the file:
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@@
   (junction (at 168.91 124.46) (diameter 0) (color 0 0 0 0)
   )
+  (junction (at 220.98 100.33) (diameter 0) (color 0 0 0 0)
+  )
   (junction (at 67.31 133.35) (diameter 0) (color 0 0 0 0)
   )
@@
   (junction (at 179.07 111.76) (diameter 0) (color 0 0 0 0)
   )
-  (junction (at 220.98 100.33) (diameter 0) (color 0 0 0 0)
-  )
   (junction (at 179.07 101.6) (diameter 0) (color 0 0 0 0)
   )
@@
     (stroke (width 0) (type default))
   )
+  (wire (pts (xy 220.98 119.38) (xy 220.98 121.92))
+    (stroke (width 0) (type default))
+  )
+  (polyline (pts (xy 274.32 142.24) (xy 274.32 97.79))
+    (stroke (width 0) (type default))
+  )
+  (wire (pts (xy 236.22 116.84) (xy 236.22 120.65))
+    (stroke (width 0) (type default))
+  )
+  (wire (pts (xy 184.15 68.58) (xy 184.15 72.39))
+    (stroke (width 0) (type default))
+  )
+  (wire (pts (xy 36.83 52.07) (xy 39.37 52.07))
+    (stroke (width 0) (type default))
+  )
+  (wire (pts (xy 168.91 63.5) (xy 170.18 63.5))
+    (stroke (width 0) (type default))
+  )
+  (wire (pts (xy 218.44 39.37) (xy 220.98 39.37))
+    (stroke (width 0) (type default))
+  )
+  (wire (pts (xy 39.37 60.96) (xy 39.37 59.69))
+    (stroke (width 0) (type default))
+  )
   (wire (pts (xy 236.22 106.68) (xy 236.22 100.33))
     (stroke (width 0) (type default))
   )
-  (wire (pts (xy 220.98 119.38) (xy 220.98 121.92))
-    (stroke (width 0) (type default))
-  )
-  (polyline (pts (xy 274.32 142.24) (xy 274.32 97.79))
-    (stroke (width 0) (type default))
-  )
-  (wire (pts (xy 184.15 68.58) (xy 184.15 72.39))
-    (stroke (width 0) (type default))
-  )
-  (wire (pts (xy 36.83 52.07) (xy 39.37 52.07))
-    (stroke (width 0) (type default))
-  )
-  (wire (pts (xy 168.91 63.5) (xy 170.18 63.5))
-    (stroke (width 0) (type default))
-  )
-  (wire (pts (xy 218.44 39.37) (xy 220.98 39.37))
-    (stroke (width 0) (type default))
-  )
-  (wire (pts (xy 39.37 60.96) (xy 39.37 59.69))
-    (stroke (width 0) (type default))
-  )
   (wire (pts (xy 236.22 45.72) (xy 236.22 39.37))
     (stroke (width 0) (type default))
@@
     (stroke (width 0) (type default))
   )
+  (wire (pts (xy 236.22 120.65) (xy 238.76 120.65))
+    (stroke (width 0) (type default))
+  )
   (wire (pts (xy 67.31 133.35) (xy 72.39 133.35))
     (stroke (width 0) (type default))
@@
     (stroke (width 0) (type default))
   )
-  (wire (pts (xy 236.22 120.65) (xy 238.76 120.65))
-    (stroke (width 0) (type default))
-  )
   (wire (pts (xy 162.56 119.38) (xy 162.56 111.76))
     (stroke (width 0) (type default))
@@
     (stroke (width 0) (type default))
   )
-  (wire (pts (xy 236.22 116.84) (xy 236.22 120.65))
-    (stroke (width 0) (type default))
-  )
   (wire (pts (xy 67.31 116.84) (xy 67.31 120.65))
     (stroke (width 0) (type default))
@@
     (stroke (width 0) (type default))
   )
+  (wire (pts (xy 236.22 100.33) (xy 220.98 100.33))
+    (stroke (width 0) (type default))
+  )
   (wire (pts (xy 168.91 58.42) (xy 168.91 63.5))
     (stroke (width 0) (type default))
@@
   )
   (wire (pts (xy 36.83 57.15) (xy 39.37 57.15))
-    (stroke (width 0) (type default))
-  )
-  (wire (pts (xy 236.22 100.33) (xy 220.98 100.33))
     (stroke (width 0) (type default))
   )
@@
     )
   )
-  (symbol (lib_id "Transistor_FET:IRF4905") (at 233.68 111.76 0) (unit 1)
-    (in_bom yes) (on_board yes) (dnp no) (fields_autoplaced)
-    (property "Reference" "Q8" (at 240.03 110.49 0)
-      (effects (font (size 1.27 1.27)) (justify left))
-    )
-    (property "Value" "IRF4905" (at 240.03 113.03 0)
-      (effects (font (size 1.27 1.27)) (justify left))
-    )
-    (property "Footprint" "Package_TO_SOT_THT:TO-220-3_Horizontal_TabDown" (at 238.76 113.665 0)
+  (symbol (lib_id "Transistor_FET:IRF4905") (at 233.68 111.76 0) (mirror x) (unit 1)
+    (in_bom yes) (on_board yes) (dnp no)
+    (property "Reference" "Q8" (at 240.03 113.03 0)
+      (effects (font (size 1.27 1.27)) (justify left))
+    )
+    (property "Value" "IRF4905" (at 240.03 110.49 0)
+      (effects (font (size 1.27 1.27)) (justify left))
+    )
+    (property "Footprint" "Package_TO_SOT_THT:TO-220-3_Horizontal_TabDown" (at 238.76 109.855 0)
       (effects (font (size 1.27 1.27) italic) (justify left) hide)
     )
@@
     )
   )
-  (symbol (lib_id "Transistor_FET:IRF4905") (at 233.68 50.8 0) (unit 1)
-    (in_bom yes) (on_board yes) (dnp no) (fields_autoplaced)
-    (property "Reference" "Q7" (at 240.03 49.53 0)
-      (effects (font (size 1.27 1.27)) (justify left))
-    )
-    (property "Value" "IRF4905" (at 240.03 52.07 0)
-      (effects (font (size 1.27 1.27)) (justify left))
-    )
-    (property "Footprint" "Package_TO_SOT_THT:TO-220-3_Horizontal_TabDown" (at 238.76 52.705 0)
+  (symbol (lib_id "Transistor_FET:IRF4905") (at 233.68 50.8 0) (mirror x) (unit 1)
+    (in_bom yes) (on_board yes) (dnp no)
+    (property "Reference" "Q7" (at 240.03 52.07 0)
+      (effects (font (size 1.27 1.27)) (justify left))
+    )
+    (property "Value" "IRF4905" (at 240.03 49.53 0)
+      (effects (font (size 1.27 1.27)) (justify left))
+    )
+    (property "Footprint" "Package_TO_SOT_THT:TO-220-3_Horizontal_TabDown" (at 238.76 48.895 0)
       (effects (font (size 1.27 1.27) italic) (justify left) hide)
     )

Commit message: Change capacitor value.
Parts:
- C1, C2: value 100uF -> 47uF
Changed lines of the file:
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@@
       (effects (font (size 1.27 1.27)) (justify left))
     )
-    (property "Value" "100uF" (at 171.45 129.54 0)
+    (property "Value" "47uF" (at 171.45 129.54 0)
       (effects (font (size 1.27 1.27)) (justify left))
     )
@@
       (effects (font (size 1.27 1.27)) (justify left))
     )
-    (property "Value" "100uF" (at 171.45 68.58 0)
+    (property "Value" "47uF" (at 171.45 68.58 0)
       (effects (font (size 1.27 1.27)) (justify left))
     )
